Commit message: 20241129

File: my_lite6_description/urdf/lite6_robot.urdf.xacro (robot description, xacro)
@@ -19,4 +19,5 @@
   <xacro:arg name="report_type" default="normal"/>
   <xacro:arg name="ros2_control_plugin" default="uf_robot_hardware/UFRobotSystemHardware"/>
+  <!--<xacro:arg name="ros2_control_plugin" default="gazebo_ros2_control/GazeboSystem"/>-->
   <xacro:arg name="ros2_control_params" default=""/>
   <xacro:arg name="add_realsense_d435i" default="false"/>
@@ -37,5 +38,5 @@
   <xacro:arg name="baud_checkset" default="true"/>
   <xacro:arg name="default_gripper_baud" default="2000000"/>
-  <xacro:arg name="attach_to" default="xarm_link"/>
+ <xacro:arg name="attach_to" default="xarm_link"/>
   <xacro:arg name="attach_xyz" default="0 0 0"/>
   <xacro:arg name="attach_rpy" default="0 0 0"/>
@@ -75,7 +76,9 @@
   </xacro:macro>
   <xacro:macro name="box_inertia" params="m x y z">
-          <inertia  ixx="${m*(y*y+z*z)/12}" ixy = "0" ixz = "0"
-                    iyy="${m*(x*x+z*z)/12}" iyz = "0"
-                    izz="${m*(x*x+z*z)/12}" />
+      <origin rpy="0 0 0" xyz="${x/2} ${y/2} ${z/2}"/>
+      <mass value="${m}"/>
+      <inertia  ixx="${m*(y*y+z*z)/12}" ixy="0" ixz="0"
+                iyy="${m*(x*x+z*z)/12}" iyz="0"
+                izz="${m*(x*x+y*y)/12}" />
   </xacro:macro>
   <xacro:macro name="sphere_inertia" params="m r">
@@ -84,8 +87,8 @@
                     izz="${2*m*r*r/5}" />
   </xacro:macro>
-  <link name="world" />
+  <link name="world"/>
   <link name="baseplate_link">
     <visual>
-      <origin xyz="0 0 0.0" />
+      <origin xyz="0.0 0.0 0.0" />
       <geometry>
         <box size="0.7 1.1 0.03" />
@@ -94,8 +97,9 @@
     </visual>
     <inertial>
-      <mass value="10"/>
-      <xacro:box_inertia m="10" x="1.1" y="0.7" z="0.03"/>
+      <!--<origin xyz="0.35 0.5 0.0" />-->
+      <xacro:box_inertia m="20" x="0.7" y="1.1" z="0.03"/>
     </inertial>
     <collision>
+      <origin xyz="0 0 0.0" />
       <geometry>
         <box size="0.7 1.1 0.03" />
@@ -103,8 +107,9 @@
     </collision>
   </link>
+  <!-- dit is niet juist parent en child zijn omgedraaid -->
   <joint name="baseplate_joint" type="fixed">
     <origin xyz="0 0 -0.015" />
-    <parent link="world" />
-    <child link="baseplate_link" />
+    <child link="world" />
+    <parent link="baseplate_link" />
   </joint>
   <link name="mountingplate_link">
@@ -117,8 +122,8 @@
     </visual>
     <inertial>
-      <mass value="1"/>
       <xacro:box_inertia m="1" x="0.130" y="0.190" z="0.005"/>
     </inertial>
     <collision>
+      <origin xyz="0 0 0.0" />
       <geometry>
         <box size="0.13 0.19 0.005" />
@@ -131,5 +136,6 @@
     <child link="mountingplate_link" />
   </joint>
-  <link name="xarm_link"/>
+  <link name="xarm_link">
+  </link >
   <joint name="base_plate_to_xarm_joint" type="fixed">
     <origin xyz="-0.0 0.0 0.0025" />
@@ -137,5 +143,12 @@
     <child link="xarm_link" />
   </joint>
+  <gazebo reference="baseplate_link">
+    <material>Gazebo/DarkGrey</material>
+  </gazebo>
+  <gazebo reference="mountingplate_link">
+    <material>Gazebo/Red</material>
+  </gazebo>
   <!-- tool center point -->
+<!--
   <link name="tcp_link" />
   <joint name="tool_link" type="fixed">
@@ -144,7 +157,7 @@
     <origin xyz="0.0 0.0 0.0" rpy="0.0 0.0 0.0"/>
   </joint>
-<!--
-  <xacro:include filename="$(find xarm_description)/urdf/gripper/lite_gripper.urdf.xacro" />
-  <xacro:uflite_gripper_urdf prefix="$(arg prefix)" attach_to='link_eef' />
 -->
+    <gazebo reference="world">
+      <turnGravityOff>true</turnGravityOff>
+    </gazebo>
 </robot>

Commit message: 20241130

File: my_lite6_description/urdf/lite6_robot.urdf.xacro (robot description, xacro)
@@ -76,5 +76,5 @@
   </xacro:macro>
   <xacro:macro name="box_inertia" params="m x y z">
-      <origin rpy="0 0 0" xyz="${x/2} ${y/2} ${z/2}"/>
+      <origin rpy="0 0 0" xyz="0 0 ${z/2}"/>
       <mass value="${m}"/>
       <inertia  ixx="${m*(y*y+z*z)/12}" ixy="0" ixz="0"
@@ -109,7 +109,7 @@
   <!-- dit is niet juist parent en child zijn omgedraaid -->
   <joint name="baseplate_joint" type="fixed">
-    <origin xyz="0 0 -0.015" />
-    <child link="world" />
-    <parent link="baseplate_link" />
+    <origin xyz="0 0 0.015" />
+    <parent link="world" />
+    <child link="baseplate_link" />
   </joint>
   <link name="mountingplate_link">
